Commit message: feat: add PPO RL training infrastructure for Optimus walking
- optimus_env.py: Gymnasium env, 56-dim obs, 15 actuators, parallelogram via qfrc_applied
- train.py: PPO 8 parallel envs, VecNormalize, checkpoints, eval callback
- snapshot.py: offscreen MuJoCo render + Telegram photo notification per milestone
- vecnorm.pkl: saved normalisation stats from 20M-step run 1
- .gitignore: exclude large model zips and intermediate checkpoints

Run 1 result: policy plateaued at mean_r=-10 (~22 step episodes). Reward reshaping needed before run 2.

File: optimus/urdf/full/Assembly.urdf (robot description, URDF)
Before this commit: robot Assembly, 24 links, 23 joints
Links:
- link Anckle-L: mass 0.6251904951882112 -> 0.6251904951872198
- link Feet-R: mass 0.5549639900514602 -> 0.3559112386235104
